File: kicad/1581-improved.sch (KiCad schematic (older format))
At the start: 81 parts, among them CN1 IEC, CN2 FLOPPY, CN3 DIN6, CN4 DIN6, CN5 CN5, CN7 CN7, J1 DRVPWR, J2 12VDC, SW1 DS02-254-1L-02BE, SW2 300DP1J1BLKM7QE, U1 W65C02CPU-40DIP, U10 74LS93, U11 74LS07, U12 SN7406N, U13 74LS241, U14 74LVC1G08GV, U15 V7805-2000R, U2 27C512, U3 62256, U4 WD1770, U5 MOS6520, U6 74LS139, U7 74LS00, U8 SN7406N, U9 74LS14, X1 ACO-16.000MHZ-EK

Commit message: Add files via upload
Parts:
- R13: value 1k -> 150R
Changed lines of the file:
@@
 P 15000 8050
 F 0 "R13" V 14795 8050 50  0000 C CNN
-F 1 "1k" V 14886 8050 50  0000 C CNN
+F 1 "150R" V 14886 8050 50  0000 C CNN
 F 2 "Resistor_THT:R_Axial_DIN0309_L9.0mm_D3.2mm_P12.70mm_Horizontal" H 15000 8050 50  0001 C CNN
 F 3 "~" H 15000 8050 50  0001 C CNN
